File: project/Oric Tactile KB/1.3b/Oric Tactile KB 1.3b.brd (EAGLE design)
At the start: 273.1 x 146.1 mm, 63 parts, among them IC1 4051N

Commit message: Update OriClone-1.pdf, OriClone-1 v2.3.zip, OriClone-1 v2.31.zip, and 44 more files
Parts:
- moved JP1 16.4 mm to (156.8, 121.3)
Routing:
- net KB_INT: track 96.8 -> 65.1 mm, vias 1 -> 0
- net ROW_1: track 526.1 -> 503.4 mm, vias 2 -> 4
- net +5V: track 114.2 -> 97.7 mm
- net ROW_A2: track 107.0 -> 90.5 mm
- net ROW_A0: track 94.7 -> 78.2 mm
- net ROW_A1: track 100.8 -> 84.3 mm
- net COL_4: track 576.7 -> 593.2 mm
- net COL_1: track 543.2 -> 559.7 mm
- net COL_0: track 399.4 -> 415.8 mm
- net GND: track 111.6 -> 95.9 mm
- net COL_7: track 623.9 -> 611.7 mm
- net COL_3: track 604.1 -> 616.1 mm
- net ROW_6: track 453.4 -> 447.6 mm, vias 0 -> 2
- net COL_2: track 555.3 -> 550.8 mm
- net ROW_0: track 585.4 -> 588.1 mm
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Other:
- board text added: "KB Revision 1.3b (Final) With optional LED By Jennifer Gunn."
- board text removed: "KB Revision 1.2b (Centers OriClone-1 PCB) With optional LED By Jennifer Gunn."
