File: project/OriClone-1/OriClone-1.brd (EAGLE design)
At the start: 206.5 x 138 mm, 93 parts, among them IC10 W65C22, IC11 SY or R6502A, IC12 ICM7555, IC13 7805 or equivalent, IC14 LM358, IC2 74F04N, IC3 74LS257N, IC4 74LS257N, IC7 28C256_DIP, IC8 74LS00N, IC9 74LS365N, K1 351, Q1 12MHz, T1 2N3904, T2 2N3904, T3 2N3904, T5 2N3904, U1 AY-3-8912A, X1 MAB7SH

Commit message: Cumulative fixes for mistakes to earlier version
Parts:
- added C22: 100nF, rcl:C050-025X075
- moved T5 6.79 mm to (30.5, 70.8), turned to 90 degrees
- moved C5 0.64 mm to (17.8, 65.1)
- moved R17 0.32 mm to (6.99, 92.7)
- moved Q1 0.32 mm to (10.5, 40.6)
Connections:
- net +5V: now also C22.2
- net GND: now also C22.1; no longer D2.A, D3.C, IC14.3, R13.1
- net N$17: now also D2.A, D3.C, IC14.3, R13.1
Routing:
- net N$17: track 15.0 -> 44.7 mm
- net N$18: track 9.22 -> 5.55 mm
- net GND: track 1147.4 -> 1144.6 mm
- net N$20: track 25.6 -> 23.4 mm
- net I/O_CONTROL: track 158.4 -> 160.0 mm
- net +5V: track 1025.5 -> 1026.7 mm
Other:
- board text added: "Release 2.2 by Duncan Gunn."
- board text removed: "Release 1.0 by Duncan Gunn."

Commit message: The OriClone-1 has had a little cosmetic!
Also, the keyboard spacebar positioning has been fixed, and there's a new keyboard variant that centers the OriClone-1 PCB.
Parts:
- IC10: value W65C22 -> 6522A
- R36: device rcl:0207/2V -> rcl:0207/7
- U1: value AY-3-8912A -> AY-3-8912
- moved R30 9.09 mm to (135.3, 121.0), turned to 180 degrees
- moved R8 5.17 mm to (135.3, 118.1), turned to 180 degrees
- moved R36 1.31 mm to (199.1, 110.5)
- moved C25 0.64 mm to (193.0, 92.1), turned to 0 degrees
- moved R28 0.63 mm to (198.4, 33.0)
- moved S1 0.45 mm to (195.3, 101.3), turned to 270 degrees
- moved R33 0.45 mm to (37.5, 7.78)
Routing:
- net +5V: track 1026.7 -> 1009.6 mm, vias 2 -> 1
- net I/O_CONTROL: track 160.0 -> 151.3 mm
- net N$22: track 52.6 -> 59.5 mm, vias 2 -> 1
- net GND: track 1144.6 -> 1141.7 mm
- net A7: track 274.0 -> 271.5 mm
- net !NMI: track 141.2 -> 143.7 mm, vias 3 -> 4
- net A9: track 233.0 -> 235.4 mm
- net A14: track 288.3 -> 289.6 mm
- net N$17: track 44.7 -> 43.4 mm
- net A12: track 230.4 -> 231.4 mm, vias 3 -> 4
- net !ROMDIS: track 69.0 -> 68.3 mm
- net A15: track 223.9 -> 224.7 mm
- net A13: track 243.6 -> 243.0 mm
- net A11: track 209.1 -> 208.5 mm
Other:
- board text added: "Release 2.3 by Jennifer Gunn."
- board text removed: "Release 2.2 by Duncan Gunn."

Commit message: Update OriClone-1.pdf, OriClone-1 v2.3.zip, OriClone-1 v2.31.zip, and 44 more files
Parts:
- moved C22 1.59 mm to (20.3, 92.4)
- moved C26 0.95 mm to (190.5, 112.7)
- moved IC13 0.64 mm to (175.3, 104.8)
- moved R30 0.64 mm to (135.3, 121.6)
- moved R8 0.64 mm to (135.3, 118.7)
- moved R31 0.32 mm to (21.6, 23.8)
- moved R32 0.32 mm to (26.7, 23.8)
Routing:
- net KBD_COL2: track 133.3 -> 138.0 mm, vias 3 -> 2
- net PB0: track 188.4 -> 192.7 mm, vias 4 -> 3
- net !MAP: track 128.1 -> 126.0 mm
- net PHI2: track 331.2 -> 332.9 mm
- net N$22: track 59.5 -> 58.1 mm
- net KBD_COL6: track 138.8 -> 140.0 mm
- net !IRQ: track 151.2 -> 150.3 mm
- net A2: track 311.8 -> 310.9 mm
- net D3: track 275.5 -> 276.1 mm
- net A7: track 271.5 -> 272.0 mm
- net A4: track 235.6 -> 236.1 mm
- net A11: track 208.5 -> 209.0 mm
- net GND: track 1141.7 -> 1141.3 mm, vias 12 -> 11
Other:
- board text added: "Release 2.31 by Jennifer Gunn."
- board text removed: "Release 2.3 by Jennifer Gunn."

Commit message: Updated the board artwork for the OriClone 1 to v2.32, also added a slimmer keyboard layout that is easier to mount.
Parts:
- IC1: value (none) -> IC1
- R23: device rcl:0207/2V -> rcl:0207/10
- R36: device rcl:0207/7 -> rcl:0207/10
- moved R36 19.4 mm to (199.9, 91.1), turned to 270 degrees
- moved C7 4.29 mm to (92.9, 25.9)
- moved R23 1.28 mm to (104.1, 13.5)
- moved D5 0.16 mm to (164.8, 33.8)
- renumbered U1 to IC15
Routing:
- net +5V: track 1009.6 -> 1014.7 mm
- net N$19: track 14.9 -> 18.1 mm
- net A9: track 235.4 -> 232.4 mm
- net !NMI: track 143.7 -> 140.7 mm, vias 4 -> 3
- net GND: track 1141.3 -> 1139.3 mm
- net SOUND_OUT: track 156.0 -> 154.1 mm
- net D0: track 307.0 -> 305.6 mm
- net I/O_CONTROL: track 151.2 -> 150.0 mm
- net D6: track 299.5 -> 298.9 mm
- net D7: track 329.7 -> 330.3 mm
- net MA6: track 73.9 -> 73.4 mm
- net PHI2: track 332.9 -> 333.4 mm
Other:
- board text added: "HCS10017"
- board text added: "Release 2.32 by Jennifer Gunn."
- board text removed: "Release 2.31 by Jennifer Gunn."
