File: project/OriClone-1/OriClone-1.sch (EAGLE design)
At the start: 90 parts, among them IC11 SY or R6502A (2MHz part), IC12 ICM7555, IC2 74F04N, IC3 74LS257N, IC4 74LS257N, IC7 28C256_DIP, IC8 74LS00N, IC9 74LS365N, K1 351, Q1 12MHz, T1 2SC1815, T2 2SC1815, T3 2SC1815, T4 2SC1815, X1 MAB7SH

Commit message: Added amended board and new keyboard design.  Also included is pre-done gerbers and excellon drill files.
Parts:
- removed C22, C23, C24: 100nF, rcl:C-EU050-025X075
- removed T4: 2SC1815, transistor:2SC1815
- added C25: 100uF 25V 105C, rcl:CPOL-EUE2.5-7
- added C26: 100nF, rcl:C-EU050-025X075
- added D5: BAT85, diode:BAT81
- added IC13: 7805 or equivalent, linear:7805T
- added T5: 2N3904, transistor:2N3904
- added U$2: 2.1MMJACKTHM, adafruit:2.1MMJACKTHM
- C1: value (none) -> 120pF
- C2, C3, C4, C5: device rcl:C-EU050-024X044 -> rcl:C-EU050-025X075
- IC10: value (none) -> W65C22
- IC11: value SY or R6502A (2MHz part) -> SY or R6502A
- R1, R13, R2, R23, R3, R31, R32, R4, R6: device rcl:R-EU_0207/10 -> rcl:R-EU_0207/2V
- R14: device rcl:R-EU_0207/10 -> rcl:R-EU_0207/7
- R36: value 220K -> 100K; device rcl:R-EU_0207/10 -> rcl:R-EU_0207/2V
- T1, T2, T3: value 2SC1815 -> 2N3904; device transistor:2SC1815 -> transistor:2N3904
- U1: value (none) -> AY-3-8912A
- renumbered U$1 to IC14
Connections:
- removed net AGND: C6.2, R21.2, R22.2, U1.VSS
- removed net GNDA: SK1.3
- new net N$22: C25.+, IC13.VI, U$2.TIP
- new net N$25: IC8C.I0, IC8C.I1, IC8D.O
- new net N$29: D5.C, IC10.IRQB
- net !CAS: now also IC2F.O; no longer IC2C.O
- net !IRQ: now also D5.A; no longer IC10.IRQB
- net !PHI2: now also IC2C.O; no longer IC2F.O
- net !RESET: now also T1.C; no longer T4.C
- net +5V: now also C26.1, IC13.VO, IC8D.I0, IC8D.I1; no longer C22.1, C23.1, C24.1, IC5.!G, IC6.!G
- net CAS: now also IC2F.I; no longer IC2C.I
- net CB1: now also T5.C; no longer T3.C
- net GND: now also C25.-, C26.2, C6.2, IC13.GND, IC5.!G, IC6.!G, R21.2, R22.2, SK1.3, T5.E, U$2.RING, U$2.RING_SW, U1.VSS; no longer C22.2, C23.2, C24.2, T4.E
- net N$10: now also K13.S; no longer K12.S
- net N$11: now also K13.P; no longer K12.P
- net N$18: now also T5.B; no longer T3.B
- net N$26: now also T1.B; no longer T4.B
- net N$6: now also T2.B; no longer T1.B
- net N$7: now also T3.C; no longer T2.C
- net N$9: now also T3.B; no longer T2.B
- net PB3: now also T2.C; no longer T1.C
- net PHI2: now also IC2C.I; no longer IC2F.I
Other:
- note added: "It is strongly reccomended that a switching equivalent is used. Board space to provide room for either including heatsink space."
- note removed: "To add an optional reset switch, put it across C12"
- note removed: "To be dealt with later"
- moved on the sheet: C10, C11, C12, C13, IC12, IC2C, IC2F, R31, R32, R33, R34

Commit message: Cumulative fixes for mistakes to earlier version
Parts:
- added C22: 100nF, rcl:C-EU050-025X075
Connections:
- net +5V: now also C22.2
- net GND: now also C22.1; no longer D2.A, D3.C, IC14G$1.+IN, R13.1
- net N$17: now also D2.A, D3.C, IC14G$1.+IN, R13.1

Commit message: The OriClone-1 has had a little cosmetic!
Also, the keyboard spacebar positioning has been fixed, and there's a new keyboard variant that centers the OriClone-1 PCB.
Parts:
- IC10: value W65C22 -> 6522A
- R36: device rcl:R-EU_0207/2V -> rcl:R-EU_0207/7
- U1: value AY-3-8912A -> AY-3-8912
Other:
- moved on the sheet: R14

Commit message: Update OriClone-1.pdf, OriClone-1 v2.3.zip, OriClone-1 v2.31.zip, and 44 more files
Other:
- note added: "Note: No amplifier is provided. Sound must be taken from either the video port or the cassette port."
- note added: "Note: Using a W65C22S variant may require changing R20 to 270R. This is because of bus holding circuitry in the WDC part."
- note removed: "Note to self:- The tape interface will need tweaking, especially the clipping diodes."
- note removed: "Note: No amplifier is provided. Sound must be taken from either the SCART port or the Cassette Port."
- moved on the sheet: C14, C15, C9, D5, IC10, IC11, R28, R29, R30, R36, S1, SV1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

Commit message: Updated the board artwork for the OriClone 1 to v2.32, also added a slimmer keyboard layout that is easier to mount.
Parts:
- IC1: value (none) -> IC1
- R23: device rcl:R-EU_0207/2V -> rcl:R-EU_0207/10
- R36: device rcl:R-EU_0207/7 -> rcl:R-EU_0207/10
- renumbered U1 to IC15
